Commit message: minor changes

File: urdf/inc/ur_macro.xacro (robot description, xacro)
@@ -42,6 +42,6 @@
      - Muhammad Asif Rana
   -->
-  <xacro:include filename="$(find ur_description)/urdf/inc/ur_transmissions.xacro" />
-  <xacro:include filename="$(find ur_description)/urdf/inc/ur_common.xacro" />
+  <xacro:include filename="$(find ur3ehand_description)/urdf/inc/ur_transmissions.xacro" />
+  <xacro:include filename="$(find ur3ehand_description)/urdf/inc/ur_common.xacro" />
   <xacro:macro name="ur_robot" params="
     prefix

File: urdf/ur.xacro (robot description, xacro)
@@ -2,5 +2,5 @@
 <robot xmlns:xacro="http://wiki.ros.org/xacro" name="ur">
    <!-- import main macro -->
-   <xacro:include filename="$(find ur_description)/urdf/inc/ur_macro.xacro"/>
+   <xacro:include filename="$(find ur3ehand_description)/urdf/inc/ur_macro.xacro"/>
    <!-- parameters -->
    <xacro:arg name="joint_limit_params" default=""/>

File: urdf/ur3e_with_hand.urdf (robot description, URDF)
Before this commit: robot ur3e_with_hand, 12 links, 11 joints
Links:
- link base_link_inertia: geometry collision mesh filename=package://ur3ehand_description/meshes/ur3e/collision/base.s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; visual mesh filename=package://ur3ehand_description/meshes/ur3e/visual/base.dae
