Commit message: checkupdate

File: urdf/ur3e_with_hand.urdf (robot description, URDF)
Before this commit: robot ur3e_with_hand, 12 links, 11 joints
Joints:
- joint wrist_3_joint: limit lower=-6.283185307179586 upper=6.283185307179586 effort=12.0 velocity=6.283185307179586 -> lower=-0.7853981625 upper=1.570796325 effort=12.0 velocity=6.283185307179586
